Commit message: fine tune camera positioning and arm links

File: src/ur5e_isaac_moveit_config/config/ur5e.urdf.xacro (robot description, xacro)
@@ -1,5 +1,5 @@
 <?xml version="1.0"?>
 <robot xmlns:xacro="http://www.ros.org/wiki/xacro" name="ur5e">
-    <xacro:arg name="initial_positions_file" default="initial_positions.yaml" />
+    <xacro:arg name="initial_positions_file" default="$(find ur5e_isaac_moveit_config)/config/initial_positions.yaml" />
     <!-- Import ur5e urdf file -->
     <xacro:include filename="/home/sheil/Development/VLA_Arm_Controller/urdf/ur5e_isaac_sim.urdf.xacro" />

File: urdf/ur5e_isaac_sim.urdf.xacro (robot description, xacro)
@@ -1,4 +1,7 @@
 <?xml version="1.0"?>
 <robot xmlns:xacro="http://wiki.ros.org/xacro" name="ur5e">
+  <xacro:arg name="initial_positions_file" default="$(find ur5e_isaac_moveit_config)/config/initial_positions.yaml"/>
+  <xacro:property name="initial_positions_file" default="$(arg initial_positions_file)"/>
+  <xacro:property name="initial_positions" value="${xacro.load_yaml(initial_positions_file)['initial_positions']}"/>
   <xacro:include filename="$(find ur_description)/urdf/ur_macro.xacro"/>
   <xacro:include filename="$(find ur_description)/urdf/inc/ur_joint_control.xacro"/>
@@ -34,5 +37,5 @@
       <param name="joint_states_topic">/joint_states</param>
     </hardware>
-    <xacro:ur_joint_control_description tf_prefix=""/>
+    <xacro:ur_joint_control_description tf_prefix="" initial_positions="${initial_positions}"/>
     <!-- Gripper: only the actuated joint; mimic joints follow automatically -->
     <joint name="robotiq_85_left_knuckle_joint">
